File: PCB/hat/greenhouse_project_hat/Heating.kicad_sch (KiCad schematic)
At the start: 29 parts, among them J16 Screw_Terminal_01x02, Q7 IPD036N04LGATMA1

Commit message: Updated PCB files
Parts:
- removed D10: LED, LED_SMD:LED_1206_3216Metric_Pad1.42x1.75mm_HandSolder, symbol Device:LED
- removed D11: SS54, DIOM5126X245N, symbol SamacSys_Parts:SS54
- removed Q7: IPD036N04LGATMA1, IPD036N04LGATMA1, symbol SamacSys_Parts:IPD036N04LGATMA1
- removed R27: 12k, Resistor_SMD:R_1206_3216Metric_Pad1.30x1.75mm_HandSolder, symbol Device:R
- removed R28: 4.7k, Resistor_SMD:R_1206_3216Metric_Pad1.30x1.75mm_HandSolder, symbol Device:R
- added Q7: IRLZ44NSTRLPBF, IRF2804STRLPBF, symbol SamacSys_Parts:IRLZ44NSTRLPBF
- R35: renamed from R26; value 10k -> 1k
- renumbered C7 to C8, C8 to C9, J16 to J17, R18 to R27, R19 to R28, R20 to R29, R21 to R30, R22 to R31, R23 to R32, R24 to R33, R25 to R34
Connections:
- net BED_OUT: now also F3.2
- net GNDREF: now also Q7.3; no longer J17.2 (Pin_2)
- net at R35.2: now also Q7.1
- new net: J17.2 (Pin_2), Q7.2
Other:
- note added: "PME6"
- moved on the sheet: F3, J17, R35, TP1

Commit message: Update: hat V5.0
Parts:
- TP1: now left out of the parts list
Other:
- note removed: "PME6"
Changed lines of the file:
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@@
   (title_block
     (title "Greenhouse project FRDM-KL25Z hat")
-    (date "16-03-2023")
-    (rev "v4.0")
+    (date "18-03-2023")
+    (rev "v5.0")
     (company "OnlyPlants")
     (comment 1 "Author: Emiel Visser")
@@
     (effects (font (size 1.27 1.27)) (justify left bottom))
   )
-  (text "PME6" (at 195.58 66.04 0)
-    (effects (font (size 1.27 1.27)) (justify left bottom))
-  )
   (text "Thermistor for heater" (at 17.78 19.05 0)
     (effects (font (size 1.27 1.27)) (justify left bottom))
@@
   )
   (symbol (lib_id "Connector:TestPoint") (at 33.02 43.18 0) (unit 1)
-    (in_bom yes) (on_board yes) (dnp no)
+    (in_bom no) (on_board yes) (dnp no)
     (property "Reference" "TP1" (at 26.67 35.56 0)
       (effects (font (size 1.27 1.27)) (justify left))
@@
   )
   (symbol (lib_id "Connector:TestPoint") (at 184.15 39.37 90) (unit 1)
-    (in_bom yes) (on_board yes) (dnp no) (fields_autoplaced)
+    (in_bom no) (on_board yes) (dnp no) (fields_autoplaced)
     (property "Reference" "TP1" (at 180.848 34.29 90)
       (effects (font (size 1.27 1.27)))
@@
   )
   (symbol (lib_id "Connector:TestPoint") (at 33.02 93.98 0) (unit 1)
-    (in_bom yes) (on_board yes) (dnp no)
+    (in_bom no) (on_board yes) (dnp no)
     (property "Reference" "TP1" (at 24.13 87.63 0)
       (effects (font (size 1.27 1.27)) (justify left))
@@
   )
   (symbol (lib_id "Connector:TestPoint") (at 92.71 43.18 180) (unit 1)
-    (in_bom yes) (on_board yes) (dnp no) (fields_autoplaced)
+    (in_bom no) (on_board yes) (dnp no) (fields_autoplaced)
     (property "Reference" "TP1" (at 95.25 45.847 0)
       (effects (font (size 1.27 1.27)) (justify right))
@@
   )
   (symbol (lib_id "Connector:TestPoint") (at 92.71 93.98 180) (unit 1)
-    (in_bom yes) (on_board yes) (dnp no) (fields_autoplaced)
+    (in_bom no) (on_board yes) (dnp no) (fields_autoplaced)
     (property "Reference" "TP1" (at 95.25 96.647 0)
       (effects (font (size 1.27 1.27)) (justify right))

Commit message: First production version
Parts:
- removed C8, C9: 0.1uF, Capacitor_SMD:C_1206_3216Metric_Pad1.33x1.80mm_HandSolder, symbol Device:C
- removed D8, D9: BAV99, Package_TO_SOT_SMD:SOT-23, symbol Diode:BAV99
- removed R28: 4.7k, Resistor_SMD:R_1206_3216Metric_Pad1.30x1.75mm_HandSolder, symbol Device:R
- removed R30, R31, R32: 2.37k 1%, Resistor_SMD:R_1206_3216Metric_Pad1.30x1.75mm_HandSolder, symbol Device:R
- removed R33, R34: 0, Resistor_SMD:R_1206_3216Metric_Pad1.30x1.75mm_HandSolder, symbol Device:R
- removed RV2, RV3: R_Potentiometer, Potentiometer_THT:Potentiometer_Bourns_3296W_Vertical, symbol Device:R_Potentiometer
- Q7: footprint IRF2804STRLPBF -> SamacSys_Parts:IRF2804STRLPBF
- R28: renamed from R27; value 4.7k -> 100k
- R29: value 2.37k 1% -> 100k
- TP1: now in the parts list
- renumbered R35 to R30
Connections:
- net +3.3V: now also J?.1 (Pin_1), J?.1 (Pin_1), TP1.1, TP1.1; no longer R28.1
- net GNDREF: now also R28.2, R29.2; no longer J?.2 (Pin_2), J?.2 (Pin_2)
- net THERM1: now also J?.2 (Pin_2), R28.1
- net THERM2: now also J?.2 (Pin_2), R29.1
Other:
- note added: "PME6"
- moved on the sheet: R28, TP1
