File: PCB/hat/greenhouse_project_hat/Humidifier.kicad_sch (KiCad schematic)
At the start: 5 parts, among them J10 Conn_01x04_Socket, J9 Conn_01x02_Socket, Q3 DMN6040SVT-7

Commit message: Updated PCB files
Parts:
- removed J9: Conn_01x02_Socket, Connector_JST:JST_PH_B2B-PH-K_1x02_P2.00mm_Vertical, symbol Connector:Conn_01x02_Socket
- added J25: Conn_01x03_Socket, Connector_JST:JST_PH_B3B-PH-K_1x03_P2.00mm_Vertical, symbol Connector:Conn_01x03_Socket
- added R?: 4.7k, Resistor_SMD:R_1206_3216Metric_Pad1.30x1.75mm_HandSolder, symbol Device:R
Connections:
- net +5V: now also J25.1 (Pin_1), R?.2
- net GNDREF: now also J25.2 (Pin_2)
- net MIST-: now also J25.3 (Pin_3), R?.1
Other:
- moved on the sheet: TP1

Commit message: Update: hat V5.0
Parts:
- TP1: now left out of the parts list
Changed lines of the file:
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@@
   (title_block
     (title "Greenhouse project FRDM-KL25Z hat")
-    (date "16-03-2023")
-    (rev "v4.0")
+    (date "18-03-2023")
+    (rev "v5.0")
     (company "OnlyPlants")
     (comment 1 "Author: Emiel Visser")
@@
   )
   (symbol (lib_id "Connector:TestPoint") (at 121.92 95.25 90) (unit 1)
-    (in_bom yes) (on_board yes) (dnp no)
+    (in_bom no) (on_board yes) (dnp no)
     (property "Reference" "TP1" (at 115.57 90.17 90)
       (effects (font (size 1.27 1.27)))

Commit message: First production version
Parts:
- Q3: footprint SOT95P280X90-6N -> SamacSys_Parts:SOT95P280X90-6N
- TP1: now in the parts list
- renumbered J25 to J9
Changed lines of the file:
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@@
   (title_block
     (title "Greenhouse project FRDM-KL25Z hat")
-    (date "18-03-2023")
-    (rev "v5.0")
+    (date "16-03-2023")
+    (rev "v4.0")
     (company "OnlyPlants")
     (comment 1 "Author: Emiel Visser")
@@
   (symbol (lib_id "power:+5V") (at 107.95 77.47 0) (unit 1)
     (in_bom yes) (on_board yes) (dnp no) (fields_autoplaced)
-    (property "Reference" "#PWR089" (at 107.95 81.28 0)
+    (property "Reference" "#PWR048" (at 107.95 81.28 0)
       (effects (font (size 1.27 1.27)) hide)
     )
@@
       (project "greenhouse_project_hat"
         (path "/b27d5451-0104-43eb-badd-cec4b3afa639/4d8eb8bd-7658-4ee1-a9bd-e11f7f5e7e34"
-          (reference "#PWR089") (unit 1)
+          (reference "#PWR048") (unit 1)
         )
       )
@@
   (symbol (lib_id "Connector:Conn_01x03_Socket") (at 133.35 85.09 0) (unit 1)
     (in_bom yes) (on_board yes) (dnp no)
-    (property "Reference" "J25" (at 139.7 87.63 0)
+    (property "Reference" "J9" (at 139.7 87.63 0)
       (effects (font (size 1.27 1.27)) (justify left))
     )
@@
       (project "greenhouse_project_hat"
         (path "/b27d5451-0104-43eb-badd-cec4b3afa639/4d8eb8bd-7658-4ee1-a9bd-e11f7f5e7e34"
-          (reference "J25") (unit 1)
+          (reference "J9") (unit 1)
         )
       )
@@
   (symbol (lib_id "power:+5V") (at 121.92 77.47 0) (unit 1)
     (in_bom yes) (on_board yes) (dnp no) (fields_autoplaced)
-    (property "Reference" "#PWR048" (at 121.92 81.28 0)
+    (property "Reference" "#PWR049" (at 121.92 81.28 0)
       (effects (font (size 1.27 1.27)) hide)
     )
@@
       (project "greenhouse_project_hat"
         (path "/b27d5451-0104-43eb-badd-cec4b3afa639/4d8eb8bd-7658-4ee1-a9bd-e11f7f5e7e34"
-          (reference "#PWR048") (unit 1)
+          (reference "#PWR049") (unit 1)
         )
       )
@@
   (symbol (lib_id "power:+5V") (at 184.15 83.82 0) (unit 1)
     (in_bom yes) (on_board yes) (dnp no) (fields_autoplaced)
-    (property "Reference" "#PWR051" (at 184.15 87.63 0)
+    (property "Reference" "#PWR053" (at 184.15 87.63 0)
       (effects (font (size 1.27 1.27)) hide)
     )
@@
       (project "greenhouse_project_hat"
         (path "/b27d5451-0104-43eb-badd-cec4b3afa639/4d8eb8bd-7658-4ee1-a9bd-e11f7f5e7e34"
-          (reference "#PWR051") (unit 1)
+          (reference "#PWR053") (unit 1)
         )
       )
@@
         )
         (path "/b27d5451-0104-43eb-badd-cec4b3afa639/4d8eb8bd-7658-4ee1-a9bd-e11f7f5e7e34"
-          (reference "R41") (unit 1)
+          (reference "R22") (unit 1)
         )
       )
@@
         )
         (path "/b27d5451-0104-43eb-badd-cec4b3afa639/4d8eb8bd-7658-4ee1-a9bd-e11f7f5e7e34"
-          (reference "#PWR049") (unit 1)
+          (reference "#PWR051") (unit 1)
         )
       )
@@
   (symbol (lib_id "power:GNDREF") (at 167.64 97.79 0) (unit 1)
     (in_bom yes) (on_board yes) (dnp no) (fields_autoplaced)
-    (property "Reference" "#PWR050" (at 167.64 104.14 0)
+    (property "Reference" "#PWR052" (at 167.64 104.14 0)
       (effects (font (size 1.27 1.27)) hide)
     )
@@
       (project "greenhouse_project_hat"
         (path "/b27d5451-0104-43eb-badd-cec4b3afa639/4d8eb8bd-7658-4ee1-a9bd-e11f7f5e7e34"
-          (reference "#PWR050") (unit 1)
+          (reference "#PWR052") (unit 1)
         )
       )
@@
         )
         (path "/b27d5451-0104-43eb-badd-cec4b3afa639/4d8eb8bd-7658-4ee1-a9bd-e11f7f5e7e34"
-          (reference "#PWR090") (unit 1)
+          (reference "#PWR050") (unit 1)
         )
       )
@@
   )
   (symbol (lib_id "Connector:TestPoint") (at 121.92 95.25 90) (unit 1)
-    (in_bom no) (on_board yes) (dnp no)
+    (in_bom yes) (on_board yes) (dnp no)
     (property "Reference" "TP1" (at 115.57 90.17 90)
       (effects (font (size 1.27 1.27)))
@@
       (effects (font (size 1.27 1.27)))
     )
-    (property "Footprint" "SOT95P280X90-6N" (at 130.81 106.68 0)
+    (property "Footprint" "SamacSys_Parts:SOT95P280X90-6N" (at 130.81 106.68 0)
       (effects (font (size 1.27 1.27)) (justify left) hide)
     )
