File: PCB/hat/greenhouse_project_hat/Lights.kicad_sch (KiCad schematic)
At the start: 18 parts, among them J11 Conn_01x03_Pin, J13 Conn_01x02_Socket, J3 Screw_Terminal_01x02, Q19 IRLZ44NSTRLPBF

Commit message: Updated PCB files
Parts:
- renumbered J13 to J14, R13 to R22, R14 to R23, R15 to R24, R16 to R25

Commit message: Update: hat V5.0
Parts:
- J11, TP1: now left out of the parts list
Other:
- moved on the sheet: TP1
Changed lines of the file:
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@@
   (title_block
     (title "Greenhouse project FRDM-KL25Z hat")
-    (date "16-03-2023")
-    (rev "v4.0")
+    (date "18-03-2023")
+    (rev "v5.0")
     (company "OnlyPlants")
     (comment 1 "Author: Emiel Visser")
@@
   (junction (at 214.63 87.63) (diameter 0) (color 0 0 0 0)
   )
+  (junction (at 121.92 91.44) (diameter 0) (color 0 0 0 0)
+  )
   (junction (at 120.65 101.6) (diameter 0) (color 0 0 0 0)
   )
@@
   (junction (at 214.63 90.17) (diameter 0) (color 0 0 0 0)
   )
-  (junction (at 125.73 91.44) (diameter 0) (color 0 0 0 0)
-  )
   (junction (at 210.82 87.63) (diameter 0) (color 0 0 0 0)
   )
@@
     (stroke (width 0) (type default))
   )
-  (wire (pts (xy 111.76 99.06) (xy 111.76 96.52))
-    (stroke (width 0) (type default))
-  )
   (wire (pts (xy 121.92 82.55) (xy 132.08 82.55))
     (stroke (width 0) (type default))
@@
     (stroke (width 0) (type default))
   )
-  (wire (pts (xy 119.38 91.44) (xy 125.73 91.44))
+  (wire (pts (xy 119.38 91.44) (xy 121.92 91.44))
     (stroke (width 0) (type default))
   )
@@
     (stroke (width 0) (type default))
   )
+  (wire (pts (xy 121.92 91.44) (xy 130.81 91.44))
+    (stroke (width 0) (type default))
+  )
   (wire (pts (xy 121.92 82.55) (xy 121.92 81.28))
     (stroke (width 0) (type default))
@@
   )
   (wire (pts (xy 228.6 92.71) (xy 228.6 90.17))
-    (stroke (width 0) (type default))
-  )
-  (wire (pts (xy 130.81 91.44) (xy 125.73 91.44))
     (stroke (width 0) (type default))
   )
@@
   )
   (symbol (lib_id "Connector:TestPoint") (at 102.87 93.98 0) (unit 1)
-    (in_bom yes) (on_board yes) (dnp no) (fields_autoplaced)
+    (in_bom no) (on_board yes) (dnp no) (fields_autoplaced)
     (property "Reference" "TP1" (at 105.41 90.043 0)
       (effects (font (size 1.27 1.27)) (justify left))
@@
   )
   (symbol (lib_id "Connector:Conn_01x03_Pin") (at 119.38 76.2 270) (unit 1)
-    (in_bom yes) (on_board yes) (dnp no) (fields_autoplaced)
+    (in_bom no) (on_board yes) (dnp no) (fields_autoplaced)
     (property "Reference" "J11" (at 119.38 72.39 90)
       (effects (font (size 1.27 1.27)))
@@
   )
   (symbol (lib_id "Connector:TestPoint") (at 120.65 101.6 0) (unit 1)
-    (in_bom yes) (on_board yes) (dnp no) (fields_autoplaced)
+    (in_bom no) (on_board yes) (dnp no) (fields_autoplaced)
     (property "Reference" "TP1" (at 123.19 97.663 0)
       (effects (font (size 1.27 1.27)) (justify left))
@@
     )
   )
-  (symbol (lib_id "Connector:TestPoint") (at 111.76 96.52 0) (unit 1)
-    (in_bom yes) (on_board yes) (dnp no) (fields_autoplaced)
-    (property "Reference" "TP1" (at 114.3 92.583 0)
-      (effects (font (size 1.27 1.27)) (justify left))
-    )
-    (property "Value" "TestPoint" (at 114.3 95.123 0)
-      (effects (font (size 1.27 1.27)) (justify left))
-    )
-    (property "Footprint" "TestPoint:TestPoint_Pad_D2.0mm" (at 116.84 96.52 0)
-      (effects (font (size 1.27 1.27)) hide)
-    )
-    (property "Datasheet" "~" (at 116.84 96.52 0)
+  (symbol (lib_id "Connector:TestPoint") (at 111.76 99.06 0) (unit 1)
+    (in_bom no) (on_board yes) (dnp no) (fields_autoplaced)
+    (property "Reference" "TP1" (at 114.3 95.123 0)
+      (effects (font (size 1.27 1.27)) (justify left))
+    )
+    (property "Value" "TestPoint" (at 114.3 97.663 0)
+      (effects (font (size 1.27 1.27)) (justify left))
+    )
+    (property "Footprint" "TestPoint:TestPoint_Pad_D2.0mm" (at 116.84 99.06 0)
+      (effects (font (size 1.27 1.27)) hide)
+    )
+    (property "Datasheet" "~" (at 116.84 99.06 0)
       (effects (font (size 1.27 1.27)) hide)
     )
@@
     )
   )
-  (symbol (lib_id "Connector:TestPoint") (at 125.73 91.44 0) (unit 1)
-    (in_bom yes) (on_board yes) (dnp no) (fields_autoplaced)
-    (property "Reference" "TP1" (at 128.27 87.503 0)
-      (effects (font (size 1.27 1.27)) (justify left))
-    )
-    (property "Value" "TestPoint" (at 128.27 90.043 0)
-      (effects (font (size 1.27 1.27)) (justify left))
-    )
-    (property "Footprint" "TestPoint:TestPoint_Pad_D2.0mm" (at 130.81 91.44 0)
-      (effects (font (size 1.27 1.27)) hide)
-    )
-    (property "Datasheet" "~" (at 130.81 91.44 0)
+  (symbol (lib_id "Connector:TestPoint") (at 121.92 91.44 0) (unit 1)
+    (in_bom no) (on_board yes) (dnp no) (fields_autoplaced)
+    (property "Reference" "TP1" (at 124.46 87.503 0)
+      (effects (font (size 1.27 1.27)) (justify left))
+    )
+    (property "Value" "TestPoint" (at 124.46 90.043 0)
+      (effects (font (size 1.27 1.27)) (justify left))
+    )
+    (property "Footprint" "TestPoint:TestPoint_Pad_D2.0mm" (at 127 91.44 0)
+      (effects (font (size 1.27 1.27)) hide)
+    )
+    (property "Datasheet" "~" (at 127 91.44 0)
       (effects (font (size 1.27 1.27)) hide)
     )
@@
   )
   (symbol (lib_id "Connector:TestPoint") (at 210.82 87.63 0) (unit 1)
-    (in_bom yes) (on_board yes) (dnp no)
+    (in_bom no) (on_board yes) (dnp no)
     (property "Reference" "TP1" (at 215.9 83.82 0)
       (effects (font (size 1.27 1.27)) (justify left))

Commit message: First production version
Parts:
- J11, TP1: now in the parts list
- Q19: footprint IRF2804STRLPBF -> SamacSys_Parts:IRF2804STRLPBF
- renumbered R22 to R23, R23 to R24, R24 to R25, R25 to R26
Other:
- moved on the sheet: TP1
