File: PCB/hat/greenhouse_project_hat/Water.kicad_sch (KiCad schematic)
At the start: 17 parts, among them J18 Screw_Terminal_01x02, Q9 DMN6040SVT-7

Commit message: Updated PCB files
Parts:
- removed D12: 1N4007, Diode_SMD:D_2512_6332Metric_Pad1.52x3.35mm_HandSolder, symbol Diode:1N4007
- added D10: RS2MA-13-F, DIOM5226X230N, symbol SamacSys_Parts:RS2MA-13-F
- renumbered J18 to J19, R29 to R36
Connections:
- net Pump+: now also D10.1
- net Pump-: now also D10.2
Other:
- moved on the sheet: TP1

Commit message: Update: hat V5.0
Parts:
- JP1, TP1: now left out of the parts list
Changed lines of the file:
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@@
   (title_block
     (title "Greenhouse project FRDM-KL25Z hat")
-    (date "16-03-2023")
-    (rev "v4.0")
+    (date "18-03-2023")
+    (rev "v5.0")
     (company "OnlyPlants")
     (comment 1 "Author: Emiel Visser")
@@
   )
   (symbol (lib_id "Connector:TestPoint") (at 238.76 67.31 270) (unit 1)
-    (in_bom yes) (on_board yes) (dnp no)
+    (in_bom no) (on_board yes) (dnp no)
     (property "Reference" "TP1" (at 254 58.42 90)
       (effects (font (size 1.27 1.27)) (justify left))
@@
   )
   (symbol (lib_id "Connector:TestPoint") (at 233.68 69.85 90) (unit 1)
-    (in_bom yes) (on_board yes) (dnp no)
+    (in_bom no) (on_board yes) (dnp no)
     (property "Reference" "TP1" (at 217.17 63.5 90)
       (effects (font (size 1.27 1.27)))
@@
   )
   (symbol (lib_id "Connector:TestPoint") (at 246.38 74.93 270) (unit 1)
-    (in_bom yes) (on_board yes) (dnp no)
+    (in_bom no) (on_board yes) (dnp no)
     (property "Reference" "TP1" (at 254 74.295 90)
       (effects (font (size 1.27 1.27)) (justify left))
@@
   )
   (symbol (lib_id "Connector:TestPoint") (at 243.84 72.39 270) (unit 1)
-    (in_bom yes) (on_board yes) (dnp no)
+    (in_bom no) (on_board yes) (dnp no)
     (property "Reference" "TP1" (at 254 68.58 90)
       (effects (font (size 1.27 1.27)) (justify left))
@@
   )
   (symbol (lib_id "Connector:TestPoint") (at 130.81 66.04 90) (unit 1)
-    (in_bom yes) (on_board yes) (dnp no) (fields_autoplaced)
+    (in_bom no) (on_board yes) (dnp no) (fields_autoplaced)
     (property "Reference" "TP1" (at 127.508 60.96 90)
       (effects (font (size 1.27 1.27)))
@@
   )
   (symbol (lib_id "Jumper:Jumper_3_Bridged12") (at 152.4 35.56 0) (unit 1)
-    (in_bom yes) (on_board yes) (dnp no) (fields_autoplaced)
+    (in_bom no) (on_board yes) (dnp no) (fields_autoplaced)
     (property "Reference" "JP1" (at 152.4 30.48 0)
       (effects (font (size 1.27 1.27)))
@@
   )
   (symbol (lib_id "Connector:TestPoint") (at 231.14 72.39 90) (unit 1)
-    (in_bom yes) (on_board yes) (dnp no)
+    (in_bom no) (on_board yes) (dnp no)
     (property "Reference" "TP1" (at 217.17 68.58 90)
       (effects (font (size 1.27 1.27)))
@@
   )
   (symbol (lib_id "Connector:TestPoint") (at 236.22 67.31 90) (unit 1)
-    (in_bom yes) (on_board yes) (dnp no)
+    (in_bom no) (on_board yes) (dnp no)
     (property "Reference" "TP1" (at 217.17 58.42 90)
       (effects (font (size 1.27 1.27)))
@@
   )
   (symbol (lib_id "Connector:TestPoint") (at 152.4 48.26 90) (unit 1)
-    (in_bom yes) (on_board yes) (dnp no) (fields_autoplaced)
+    (in_bom no) (on_board yes) (dnp no) (fields_autoplaced)
     (property "Reference" "TP1" (at 149.098 43.18 90)
       (effects (font (size 1.27 1.27)))
@@
   )
   (symbol (lib_id "Connector:TestPoint") (at 228.6 74.93 90) (unit 1)
-    (in_bom yes) (on_board yes) (dnp no)
+    (in_bom no) (on_board yes) (dnp no)
     (property "Reference" "TP1" (at 217.17 73.66 90)
       (effects (font (size 1.27 1.27)))
@@
   )
   (symbol (lib_id "Connector:TestPoint") (at 241.3 69.85 270) (unit 1)
-    (in_bom yes) (on_board yes) (dnp no)
+    (in_bom no) (on_board yes) (dnp no)
     (property "Reference" "TP1" (at 254 63.5 90)
       (effects (font (size 1.27 1.27)) (justify left))

Commit message: First production version
Parts:
- added TP1: TestPoint, TestPoint:TestPoint_Pad_D2.0mm, symbol Connector:TestPoint
- D8: renamed from D10; footprint DIOM5226X230N -> SamacSys_Parts:DIOM5226X230N
- JP1, TP1: now in the parts list
- Q9: footprint SOT95P280X90-6N -> SamacSys_Parts:SOT95P280X90-6N
- renumbered R36 to R31
Connections:
- net +5V: now also J?.10 (Pin_10), TP1.1
- no-connect marks 1 -> 0
