File: PCB/hat/greenhouse_project_hat/greenhouse_project_hat.kicad_pcb (KiCad board)
At the start: 4 copper layers, 134 x 145.7 mm, 169 parts, among them IC1 74HCT365D,652, IC2 74HCT365D,652, J1 Conn_01x10_Socket, J11 Conn_01x03_Pin, J13 Conn_01x02_Socket, J14 Conn_01x02_Socket, J14 Screw_Terminal_01x02, J15 Conn_01x02_Socket, J18 Screw_Terminal_01x02, J19 Conn_01x10_Socket, J2 Conn_01x06_Socket, J20 Conn_01x02_Socket, J21 Conn_01x02_Socket, J22 Conn_01x02_Socket, J23 Conn_01x02_Socket, J24 Screw_Terminal_01x02, J25 Screw_Terminal_01x02, J3 Screw_Terminal_01x02, J4 Conn_01x04_Socket, J5 Conn_01x06_Pin, J6 Conn_01x06_Pin, J7 Conn_01x06_Pin, J8 Conn_01x06_Pin, J9 Conn_01x02_Socket, Q1 RZF030P01, Q10 DMN6040SVT-7, Q11 DMN6040SVT-7, Q12 DMN6040SVT-7, Q2 AO3401A, Q3 DMN6040SVT-7, Q4 IRLZ44NSTRLPBF, Q5 IRLZ44NSTRLPBF, Q6 IRLZ44NSTRLPBF, Q7 IPD036N04LGATMA1, Q8 DMN6040SVT-7, Q9 DMN6040SVT-7, SW1 TestPoint, SW2 TestPoint, SW3 TestPoint, SW4 TestPoint, SW5 TestPoint, U1 LM2596 Buck

Commit message: Updated PCB files
Parts:
- removed 2-, 3-, 4-: TestPoint, TestPoint:TestPoint_Pad_D2.0mm
- removed D15, D16: 1N4007, Diode_SMD:D_2512_6332Metric_Pad1.52x3.35mm_HandSolder
- removed J9: Conn_01x02_Socket, Connector_JST:JST_PH_B2B-PH-K_1x02_P2.00mm_Vertical
- removed the R28 at (187.7, 131.4)
- added J25: Conn_01x03_Socket, Connector_JST:JST_PH_B3B-PH-K_1x03_P2.00mm_Vertical, F.Cu at (289.6, 214.0)
- added R41: 4.7k, Resistor_SMD:R_1206_3216Metric_Pad1.30x1.75mm_HandSolder, F.Cu at (287.0, 208.3)
- added TP35: TestPoint, TestPoint:TestPoint_Pad_D2.0mm, B.Cu at (255.3, 210.5)
- added TP38: TestPoint, TestPoint:TestPoint_Pad_D2.0mm, B.Cu at (266.7, 210.5)
- added TP39: TestPoint, TestPoint:TestPoint_Pad_D2.0mm, B.Cu at (243.0, 210.5)
- D10: value LED -> RS2MA-13-F; footprint LED_SMD:LED_1206_3216Metric_Pad1.42x1.75mm_HandSolder -> SamacSys_Parts:DIOM5226X230N
- D11: value SS54 -> RS2MA-13-F; footprint SamacSys_Parts:DIOM5126X245N -> SamacSys_Parts:DIOM5226X230N
- D12, D13, D14: value 1N4007 -> RS2MA-13-F; footprint Diode_SMD:D_2512_6332Metric_Pad1.52x3.35mm_HandSolder -> SamacSys_Parts:DIOM5226X230N
- D6: value 1N4007 -> D_Schottky; footprint Diode_SMD:D_2512_6332Metric_Pad1.52x3.35mm_HandSolder -> Diode_THT:D_A-405_P10.16mm_Horizontal
- Q7: value IPD036N04LGATMA1 -> IRLZ44NSTRLPBF; footprint SamacSys_Parts:IPD036N04LGATMA1 -> SamacSys_Parts:IRF2804STRLPBF
- R35: renamed from R26; value 10k -> 1k
- moved D10 124.6 mm to (290.2, 194.3), turned to 90 degrees
- moved D11 114.7 mm to (276.2, 207.0), turned to 0 degrees
- moved D12 39.5 mm to (253.1, 207.0), turned to 0 degrees
- moved D14 12.1 mm to (240.7, 207.0)
- moved D13 12.0 mm to (264.2, 207.0)
- moved R27 10.4 mm to (200.7, 129.3)
- moved R35 10.4 mm to (200.7, 134.3)
- moved F3 8.26 mm to (187.3, 132.7)
- moved C7 7.77 mm to (271.8, 87.5)
- moved D6 6.69 mm to (279.4, 90.8)
- moved Q7 2.56 mm to (193.8, 144.1), turned to 90 degrees
- moved Q3 1.91 mm to (285.1, 204.2)
- moved R21 1.91 mm to (290.2, 204.2)
- moved R18 0.13 mm to (268.6, 106.3)
- renumbered C9 to C2, C2 to C3, C3 to C4, C4 to C7, C7 to C8, C8 to C9, RX to D1, TX to D2, AHT21b to J10, J24 to J12, J25 to J13, J13 to J14, J14 to J15, J15 to J16, J14 to J17, SOIL to J18, J18 to J19, J19 to J20, J20 to J21, J21 to J22, J22 to J23, J23 to J24, BT_RX to JP1, BT_TX to JP2, PUMP to JP3, FAN1 to JP4, FAN2 to JP5, FAN3 to JP6, FAN4 to JP7, R44 to R10, R2 to R11, R3 to R12, R4 to R13, R5 to R14, R6 to R15, R7 to R16, R8 to R17, R9 to R18, R10 to R19, R34 to R2, R11 to R20, R12 to R21, R13 to R22, R14 to R23, R15 to R24, R16 to R25, R17 to R26, R18 to R27, R19 to R28, R20 to R29, R35 to R3, R21 to R30, R22 to R31, R23 to R32, R24 to R33, R25 to R34, R29 to R36, R30 to R37, R31 to R38, R32 to R39, R36 to R4, R33 to R40, R37 to R5, R38 to R6, R39 to R7, R40 to R8, R41 to R9, SW1 to TP1, SCL to TP10, 5v to TP11, 12v to TP12, MIST- to TP13, G to TP14, R to TP15, B to TP16, + to TP17, LDR to TP18, THERM1 to TP19, SW2 to TP2, THERM2 to TP20, THERM1 to TP21, THERM2 to TP22, BED_OUT to TP23, P- to TP24, P+ to TP25, SENS1 to TP26, SENS2 to TP27, SENS3 to TP28, SENS4 to TP29, SW3 to TP3, SENS5 to TP30, SENS6 to TP31, SENS7 to TP32, SENS8 to TP33, 1- to TP34, 1+ to TP36, 2+ to TP37, SW4 to TP4, 3+ to TP40, 4+ to TP41, SW5 to TP5, 5v to TP6, 3v3 to TP7, GND to TP8, SDA to TP9
Connections:
- D10 pad 1: /Heating/BED_OUT -> /Water/Pump+
- D10 pad 2: Net-(D10-A) -> /Water/Pump-
- D11 pad 1: Net-(D11-Pad1) -> /Fans/Fan1+
- D11 pad 2: /Heating/BED_OUT -> /Fans/Fan1-
- D12 pad 1: /Water/Pump+ -> /Fans/Fan2+
- D12 pad 2: /Water/Pump- -> /Fans/Fan2-
- D13 pad 1: /Fans/Fan1+ -> /Fans/Fan3+
- D13 pad 2: /Fans/Fan1- -> /Fans/Fan3-
- D14 pad 1: /Fans/Fan2+ -> /Fans/Fan4+
- D14 pad 2: /Fans/Fan2- -> /Fans/Fan4-
- F3 pad 2: Net-(D11-Pad1) -> /Heating/BED_OUT
- J14 pad 2: +5V -> +3.3V
- J17 pad 2: GNDREF -> Net-(J17-Pin_2)
- Q7 pad 2: /Heating/BED_OUT -> Net-(J17-Pin_2)
- U1 pad 5: GNDREF -> (no net)
- U1 pad 6: GNDREF -> (no net)
Routing:
- net Net-(Q7-Pad1): track 7.09 -> 22.6 mm
- net HEATER_IN_POW: track 39.0 -> 30.0 mm
- net +5V: track 55.4 -> 61.5 mm
- net Net-(D10-A): track 2.04 -> 0.00 mm
- net /Fans/Fan2-: track 27.9 -> 26.5 mm
- net /Fans/Fan4-: track 28.9 -> 27.6 mm
- net /Humidifier/MIST-: track 21.7 -> 22.8 mm
- net MIST_EN_POW: track 38.2 -> 37.4 mm
- net /Fans/Fan2+: track 19.1 -> 18.3 mm
- net /Fans/Fan1-: track 29.1 -> 28.4 mm
- net /Fans/Fan3-: track 28.3 -> 27.7 mm
- net Net-(Q1-Pad1): track 4.63 -> 4.09 mm
- added copper zone on F.Cu, net Net-(J17-Pin_2)
- removed copper zone on F.Cu, net Net-(D11-Pad1)
Other:
- board text added: "10A"
- board text added: "7A"
- board text added: "9A"
- board text added: "EN"
- board text removed: "4A"
- board text removed: "6A"
- board text removed: "8A"

Commit message: Update: hat V5.0
Parts:
- moved Q2 2.26 mm to (284.6, 114.9)
- moved R19 2.26 mm to (286.5, 109.2)
- moved R20 2.26 mm to (282.7, 109.2)
- moved TP20 0.63 mm to (175.3, 188.0)
Routing:
- net GNDREF: track 13.6 -> 20.5 mm, vias 2 -> 3
- net ~{12V_EN}: track 22.0 -> 19.7 mm
- net /Power/BATT_EN: track 18.3 -> 20.6 mm
- net +3.3V: track 37.6 -> 39.7 mm, vias 6 -> 5
Other:
- board text added: "+12V"
- board text added: "+5V"
- board text added: "12A"
- board text added: "3.3v"
- board text added: "8A"
- board text added: "BED OUT"
- board text added: "F1+"
- board text added: "F1-"
- board text added: "F2+"
- board text added: "F2-"
- board text added: "F3+"
- board text added: "F3-"
- board text added: "F4-"
- board text added: "M-"
- board text added: "P+"
- board text added: "P-"
- board text added: "R-THERM2"
- board text added: "RXD"
- board text added: "S1"
- board text added: "S2"
- board text added: "S3"
- board text added: "S4"
- board text added: "S5"
- board text added: "S6"
- board text added: "S7"
- board text added: "S8"
- board text added: "SW1"
- board text added: "SW2"
- board text added: "SW3"
- board text added: "SW4"
- board text added: "SW5"
- board text added: "TXD"
- board text added: "V-FAN1"
- board text added: "V-FAN2"
- board text added: "V-FAN3"
- board text added: "V-FAN4"
- board text added: "V-PUMP"
- board text removed: "7A"
- board text removed: "9A"

Commit message: First production version
Parts:
- removed C8, C9: 0.1uF, Capacitor_SMD:C_1206_3216Metric_Pad1.33x1.80mm_HandSolder
- removed the D8 at (184.3, 154.9)
- removed the D9 at (184.3, 175.0)
- removed the R27 at (181.7, 166.4)
- removed the R30 at (181.7, 179.7)
- removed the R31 at (186.8, 160.0)
- removed the R32 at (186.8, 179.7)
- removed the R33 at (186.8, 166.4)
- removed the R34 at (186.8, 186.1)
- removed RV2, RV3: R_Potentiometer, Potentiometer_THT:Potentiometer_Bourns_3296W_Vertical
- added TP34: TestPoint, TestPoint:TestPoint_Pad_D2.0mm, B.Cu at (222.9, 198.1)
- F1: footprint Fuse:Fuse_Blade_Mini_directSolder -> Fuse:Fuseholder_Blade_Mini_Keystone_3568
- R28: value 4.7k -> 100k
- R29: value 2.37k 1% -> 100k
- moved R29 24.2 mm to (183.1, 184.2), turned to 0 degrees
- moved TP4 21.7 mm to (207.0, 162.4)
- moved TP8 21.7 mm to (207.0, 167.5)
- moved TP10 21.1 mm to (203.8, 170.2)
- moved R28 21.0 mm to (182.9, 164.8), turned to 0 degrees
- moved TP2 21.0 mm to (203.8, 159.8)
- moved TP6 21.0 mm to (203.8, 164.9)
- moved J1 19.9 mm to (197.8, 159.8)
- moved TP5 19.3 mm to (194.3, 164.9)
- moved TP9 19.3 mm to (194.3, 170.0)
- moved TP1 19.3 mm to (194.3, 159.8)
- moved TP3 18.5 mm to (191.1, 162.4)
- moved TP7 18.5 mm to (191.1, 167.5)
- moved TP21 7.62 mm to (184.2, 181.0)
- moved TP22 7.62 mm to (184.3, 161.3)
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- renumbered D12 to D10, D13 to D11, D14 to D12, D10 to D8, D11 to D9, J25 to J9, R41 to R22, R22 to R23, R23 to R24, R24 to R25, R25 to R26, R26 to R27, R35 to R30, R36 to R31, R37 to R32, R38 to R33, R39 to R34, R40 to R35, TP22 to TP21, TP21 to TP22, TP34 to TP35, TP35 to TP36, TP36 to TP37, TP37 to TP38, TP38 to TP39, TP39 to TP40, TP40 to TP41, TP41 to TP42
Connections:
- FRDM1 pad D0: unconnected-(FRDM1-D0/PTA1-PadD0) -> /SW1_OUT
- FRDM1 pad D1: unconnected-(FRDM1-D1/PTA2-PadD1) -> /SW2_OUT
- FRDM1 pad D2: unconnected-(FRDM1-D2/PTD4-PadD2) -> /SW3_OUT
- FRDM1 pad D3: unconnected-(FRDM1-D3/PTA12-PadD3) -> /SW4_OUT
- FRDM1 pad D4: unconnected-(FRDM1-D4/PTA4-PadD4) -> /SW5_OUT
- FRDM1 pad D6: /SW5_OUT -> unconnected-(FRDM1-D6/PTC8-PadD6)
- FRDM1 pad PTE2: /SW1_OUT -> unconnected-(FRDM1-PadPTE2)
- FRDM1 pad PTE3: /SW2_OUT -> unconnected-(FRDM1-PadPTE3)
- FRDM1 pad PTE4: /SW3_OUT -> unconnected-(FRDM1-PadPTE4)
- FRDM1 pad PTE5: /SW4_OUT -> unconnected-(FRDM1-PadPTE5)
- J15 pad 1: Net-(J15-Pin_1) -> +3.3V
- J15 pad 2: GNDREF -> THERM1
- J16 pad 1: Net-(J16-Pin_1) -> +3.3V
- J16 pad 2: GNDREF -> THERM2
- J20 pad 10: unconnected-(J20-Pin_10-Pad10) -> +5V
- R28 pad 1: +3.3V -> THERM1
- R28 pad 2: Net-(J16-Pin_1) -> GNDREF
- R29 pad 1: Net-(J15-Pin_1) -> THERM2
- R29 pad 2: Net-(D8-K-Pad3) -> GNDREF
- TP19 pad 1: Net-(J15-Pin_1) -> +3.3V
- TP20 pad 1: Net-(J16-Pin_1) -> +3.3V
Routing:
- net +3.3V: track 39.7 -> 17.8 mm, vias 5 -> 2
- net /OLED_SDA: track 83.3 -> 101.8 mm
- net /OLED_SCL: track 83.3 -> 100.5 mm
- net Net-(J15-Pin_1): track 15.1 -> 0.00 mm
- net Net-(J16-Pin_1): track 14.7 -> 0.00 mm
- net Net-(D9-K-Pad3): track 14.2 -> 0.00 mm
- net Net-(D8-K-Pad3): track 14.2 -> 0.00 mm
- net THERM2: track 139.2 -> 128.2 mm
- net /SW1_OUT: track 67.2 -> 56.7 mm, vias 0 -> 1
- net /SW5_OUT: track 67.2 -> 76.9 mm
- net GNDREF: track 20.5 -> 11.0 mm, vias 3 -> 2
- net /SW2_OUT: track 65.6 -> 56.4 mm, vias 1 -> 3
- net THERM1: track 115.9 -> 123.3 mm
- net /SW4_OUT: track 68.7 -> 61.9 mm, vias 1 -> 2
- net +5V: track 61.5 -> 66.0 mm
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Other:
- board text added: "+12v"
- board text added: "+5v"
- board text added: "BT"
- board text added: "F4+"
- board text added: "MIST-"
- board text removed: "+12V"
- board text removed: "+5V"
- board text removed: "12A"
- board text removed: "BED OUT"
- board text removed: "M-"
- board text removed: "NC"
- board text removed: "R-THERM2"
- board text removed: "V-FAN1"
- board text removed: "V-FAN2"
- board text removed: "V-FAN3"
- board text removed: "V-FAN4"
- board text removed: "V-PUMP"
