File: PCB/hat/greenhouse_project_hat/greenhouse_project_hat.kicad_sch (KiCad schematic)
At the start: 37 parts, among them IC1 74HCT365D,652, IC2 74HCT365D,652, J2 Conn_01x06_Socket

Commit message: Update: hat V5.0
Parts:
- H1, H2, H3, H4, J2, JP1, TP1: now left out of the parts list
Changed lines of the file:
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@@
   (title_block
     (title "Greenhouse project FRDM-KL25Z hat")
-    (date "16-03-2023")
-    (rev "v4.0")
+    (date "18-03-2023")
+    (rev "v5.0")
     (company "OnlyPlants")
     (comment 1 "Author: Emiel Visser")
@@
   )
   (symbol (lib_id "Mechanical:MountingHole_Pad") (at 238.76 21.59 0) (unit 1)
-    (in_bom yes) (on_board yes) (dnp no) (fields_autoplaced)
+    (in_bom no) (on_board yes) (dnp no) (fields_autoplaced)
     (property "Reference" "H1" (at 241.3 19.685 0)
       (effects (font (size 1.27 1.27)) (justify left))
@@
   )
   (symbol (lib_id "Connector:TestPoint") (at 309.88 41.91 180) (unit 1)
-    (in_bom yes) (on_board yes) (dnp no)
+    (in_bom no) (on_board yes) (dnp no)
     (property "Reference" "TP1" (at 309.88 52.07 90)
       (effects (font (size 1.27 1.27)) (justify right))
@@
   )
   (symbol (lib_id "Connector:TestPoint") (at 320.04 41.91 180) (unit 1)
-    (in_bom yes) (on_board yes) (dnp no)
+    (in_bom no) (on_board yes) (dnp no)
     (property "Reference" "TP1" (at 320.04 52.07 90)
       (effects (font (size 1.27 1.27)) (justify right))
@@
   )
   (symbol (lib_id "Connector:TestPoint") (at 304.8 41.91 180) (unit 1)
-    (in_bom yes) (on_board yes) (dnp no)
+    (in_bom no) (on_board yes) (dnp no)
     (property "Reference" "TP1" (at 304.8 52.07 90)
       (effects (font (size 1.27 1.27)) (justify right))
@@
   )
   (symbol (lib_id "Jumper:Jumper_3_Bridged12") (at 388.62 60.96 0) (unit 1)
-    (in_bom yes) (on_board yes) (dnp no) (fields_autoplaced)
+    (in_bom no) (on_board yes) (dnp no) (fields_autoplaced)
     (property "Reference" "JP1" (at 388.62 55.88 0)
       (effects (font (size 1.27 1.27)))
@@
   )
   (symbol (lib_id "Connector:TestPoint") (at 299.72 41.91 180) (unit 1)
-    (in_bom yes) (on_board yes) (dnp no)
+    (in_bom no) (on_board yes) (dnp no)
     (property "Reference" "TP1" (at 299.72 52.07 90)
       (effects (font (size 1.27 1.27)) (justify right))
@@
   )
   (symbol (lib_id "Jumper:Jumper_3_Bridged12") (at 345.44 60.96 0) (unit 1)
-    (in_bom yes) (on_board yes) (dnp no) (fields_autoplaced)
+    (in_bom no) (on_board yes) (dnp no) (fields_autoplaced)
     (property "Reference" "JP1" (at 345.44 55.88 0)
       (effects (font (size 1.27 1.27)))
@@
   )
   (symbol (lib_id "Connector:TestPoint") (at 307.34 41.91 180) (unit 1)
-    (in_bom yes) (on_board yes) (dnp no)
+    (in_bom no) (on_board yes) (dnp no)
     (property "Reference" "TP1" (at 307.34 52.07 90)
       (effects (font (size 1.27 1.27)) (justify right))
@@
   )
   (symbol (lib_id "Connector:TestPoint") (at 314.96 41.91 180) (unit 1)
-    (in_bom yes) (on_board yes) (dnp no)
+    (in_bom no) (on_board yes) (dnp no)
     (property "Reference" "TP1" (at 314.96 52.07 90)
       (effects (font (size 1.27 1.27)) (justify right))
@@
   )
   (symbol (lib_id "Mechanical:MountingHole_Pad") (at 264.16 21.59 0) (unit 1)
-    (in_bom yes) (on_board yes) (dnp no) (fields_autoplaced)
+    (in_bom no) (on_board yes) (dnp no) (fields_autoplaced)
     (property "Reference" "H3" (at 266.7 19.685 0)
       (effects (font (size 1.27 1.27)) (justify left))
@@
   )
   (symbol (lib_id "Connector:TestPoint") (at 302.26 41.91 180) (unit 1)
-    (in_bom yes) (on_board yes) (dnp no)
+    (in_bom no) (on_board yes) (dnp no)
     (property "Reference" "TP1" (at 302.26 52.07 90)
       (effects (font (size 1.27 1.27)) (justify right))
@@
   )
   (symbol (lib_id "Connector:TestPoint") (at 317.5 41.91 180) (unit 1)
-    (in_bom yes) (on_board yes) (dnp no)
+    (in_bom no) (on_board yes) (dnp no)
     (property "Reference" "TP1" (at 317.5 52.07 90)
       (effects (font (size 1.27 1.27)) (justify right))
@@
   )
   (symbol (lib_id "Connector:TestPoint") (at 312.42 41.91 180) (unit 1)
-    (in_bom yes) (on_board yes) (dnp no)
+    (in_bom no) (on_board yes) (dnp no)
     (property "Reference" "TP1" (at 312.42 52.07 90)
       (effects (font (size 1.27 1.27)) (justify right))
@@
   )
   (symbol (lib_id "Connector:TestPoint") (at 297.18 41.91 180) (unit 1)
-    (in_bom yes) (on_board yes) (dnp no)
+    (in_bom no) (on_board yes) (dnp no)
     (property "Reference" "TP1" (at 297.18 52.07 90)
       (effects (font (size 1.27 1.27)) (justify right))
@@
   )
   (symbol (lib_id "Mechanical:MountingHole_Pad") (at 238.76 35.56 0) (unit 1)
-    (in_bom yes) (on_board yes) (dnp no) (fields_autoplaced)
+    (in_bom no) (on_board yes) (dnp no) (fields_autoplaced)
     (property "Reference" "H2" (at 241.3 33.655 0)
       (effects (font (size 1.27 1.27)) (justify left))
@@
   )
   (symbol (lib_id "Connector:Conn_01x06_Socket") (at 359.41 30.48 0) (unit 1)
-    (in_bom yes) (on_board yes) (dnp no) (fields_autoplaced)
+    (in_bom no) (on_board yes) (dnp no) (fields_autoplaced)
     (property "Reference" "J2" (at 360.68 31.115 0)
       (effects (font (size 1.27 1.27)) (justify left))
@@
   )
   (symbol (lib_id "Mechanical:MountingHole_Pad") (at 264.16 35.56 0) (unit 1)
-    (in_bom yes) (on_board yes) (dnp no) (fields_autoplaced)
+    (in_bom no) (on_board yes) (dnp no) (fields_autoplaced)
     (property "Reference" "H4" (at 266.7 33.655 0)
       (effects (font (size 1.27 1.27)) (justify left))

Commit message: First production version
Parts:
- H1, H2, H3, H4, J2, JP1, TP1: now in the parts list
- IC1, IC2: footprint 74HCT365D652 -> SamacSys_Parts:74HCT365D652
Connections:
- net SW1_OUT: now also FRDM1.D0 (D0/PTA1); no longer FRDM1.PTE2
- net SW2_OUT: now also FRDM1.D1 (D1/PTA2); no longer FRDM1.PTE3
- net SW3_OUT: now also FRDM1.D2 (D2/PTD4); no longer FRDM1.PTE4
- net SW4_OUT: now also FRDM1.D3 (D3/PTA12); no longer FRDM1.PTE5
- net SW5_OUT: now also FRDM1.D4 (D4/PTA4); no longer FRDM1.D6 (D6/PTC8)
