File: PCB/hat/greenhouse_project_hat/Power.kicad_sch (KiCad schematic)
At the start: 31 parts, among them J3 Screw_Terminal_01x02, J4 Conn_01x04_Socket, J5 Conn_01x06_Pin, J6 Conn_01x06_Pin, J7 Conn_01x06_Pin, J8 Conn_01x06_Pin, Q1 RZF030P01, Q2 AO3401A, U1 LM2596 Buck

Commit message: Updated PCB files
Parts:
- removed D9: 1N4007, Diode_SMD:D_2512_6332Metric_Pad1.52x3.35mm_HandSolder, symbol Diode:1N4007
- added D6: D_Schottky, Diode_THT:D_A-405_P10.16mm_Horizontal, symbol Device:D_Schottky
- renumbered C2 to C3, C3 to C4, C4 to C7, R4 to R13, R5 to R14, R6 to R15, R7 to R16, R8 to R17, R9 to R18, R10 to R19, R11 to R20, TP12 to TP11, TP11 to TP12
Connections:
- net +12V: now also D6.1 (K)
- net BATT_EN: now also D6.2 (A)
- net GNDREF: no longer U1.5 (GND1), U1.6 (GND2)
Other:
- moved on the sheet: C5, C6, C7, D7, TP11, TP12

Commit message: Update: hat V5.0
Parts:
- J5, J6, J7, J8, TP11, TP12: now left out of the parts list
Changed lines of the file:
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@@
   (title_block
     (title "Greenhouse project FRDM-KL25Z hat")
-    (date "16-03-2023")
-    (rev "v4.0")
+    (date "18-03-2023")
+    (rev "v5.0")
     (company "OnlyPlants")
     (comment 1 "Author: Emiel Visser")
@@
   )
   (symbol (lib_id "Connector:TestPoint") (at 106.68 39.37 0) (unit 1)
-    (in_bom yes) (on_board yes) (dnp no) (fields_autoplaced)
+    (in_bom no) (on_board yes) (dnp no) (fields_autoplaced)
     (property "Reference" "TP12" (at 109.22 35.433 0)
       (effects (font (size 1.27 1.27)) (justify left))
@@
   )
   (symbol (lib_id "Connector:TestPoint") (at 81.28 92.71 90) (unit 1)
-    (in_bom yes) (on_board yes) (dnp no)
+    (in_bom no) (on_board yes) (dnp no)
     (property "Reference" "TP11" (at 74.93 87.63 90)
       (effects (font (size 1.27 1.27)))
@@
   )
   (symbol (lib_id "Connector:Conn_01x06_Pin") (at 215.9 113.03 270) (unit 1)
-    (in_bom yes) (on_board yes) (dnp no) (fields_autoplaced)
+    (in_bom no) (on_board yes) (dnp no) (fields_autoplaced)
     (property "Reference" "J5" (at 214.63 109.22 90)
       (effects (font (size 1.27 1.27)))
@@
   )
   (symbol (lib_id "Connector:Conn_01x06_Pin") (at 246.38 113.03 270) (unit 1)
-    (in_bom yes) (on_board yes) (dnp no) (fields_autoplaced)
+    (in_bom no) (on_board yes) (dnp no) (fields_autoplaced)
     (property "Reference" "J7" (at 245.11 109.22 90)
       (effects (font (size 1.27 1.27)))
@@
   )
   (symbol (lib_id "Connector:Conn_01x06_Pin") (at 215.9 132.08 270) (unit 1)
-    (in_bom yes) (on_board yes) (dnp no) (fields_autoplaced)
+    (in_bom no) (on_board yes) (dnp no) (fields_autoplaced)
     (property "Reference" "J6" (at 214.63 128.27 90)
       (effects (font (size 1.27 1.27)))
@@
   )
   (symbol (lib_id "Connector:Conn_01x06_Pin") (at 246.38 133.35 270) (unit 1)
-    (in_bom yes) (on_board yes) (dnp no) (fields_autoplaced)
+    (in_bom no) (on_board yes) (dnp no) (fields_autoplaced)
     (property "Reference" "J8" (at 245.11 129.54 90)
       (effects (font (size 1.27 1.27)))

Commit message: First production version
Parts:
- F1: footprint Fuse:Fuse_Blade_Mini_directSolder -> Fuse:Fuseholder_Blade_Mini_Keystone_3568
- J5, J6, J7, J8, TP11, TP12: now in the parts list
- Q1: footprint 2SB1730 -> SamacSys_Parts:2SB1730
Changed lines of the file:
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@@
   (title_block
     (title "Greenhouse project FRDM-KL25Z hat")
-    (date "18-03-2023")
-    (rev "v5.0")
+    (date "16-03-2023")
+    (rev "v4.0")
     (company "OnlyPlants")
     (comment 1 "Author: Emiel Visser")
@@
   )
   (symbol (lib_id "Connector:TestPoint") (at 106.68 39.37 0) (unit 1)
-    (in_bom no) (on_board yes) (dnp no) (fields_autoplaced)
+    (in_bom yes) (on_board yes) (dnp no) (fields_autoplaced)
     (property "Reference" "TP12" (at 109.22 35.433 0)
       (effects (font (size 1.27 1.27)) (justify left))
@@
   )
   (symbol (lib_id "Connector:TestPoint") (at 81.28 92.71 90) (unit 1)
-    (in_bom no) (on_board yes) (dnp no)
+    (in_bom yes) (on_board yes) (dnp no)
     (property "Reference" "TP11" (at 74.93 87.63 90)
       (effects (font (size 1.27 1.27)))
@@
       (effects (font (size 1.27 1.27)))
     )
-    (property "Footprint" "Fuse:Fuse_Blade_Mini_directSolder" (at 36.83 41.148 90)
+    (property "Footprint" "Fuse:Fuseholder_Blade_Mini_Keystone_3568" (at 36.83 41.148 90)
       (effects (font (size 1.27 1.27)) hide)
     )
@@
   (symbol (lib_id "power:GNDREF") (at 81.28 111.76 0) (unit 1)
     (in_bom yes) (on_board yes) (dnp no) (fields_autoplaced)
-    (property "Reference" "#PWR036" (at 81.28 118.11 0)
+    (property "Reference" "#PWR035" (at 81.28 118.11 0)
       (effects (font (size 1.27 1.27)) hide)
     )
@@
       (project "greenhouse_project_hat"
         (path "/b27d5451-0104-43eb-badd-cec4b3afa639/a0f75671-40a3-4d36-8542-9696f27b0c1b"
-          (reference "#PWR036") (unit 1)
+          (reference "#PWR035") (unit 1)
         )
       )
@@
       (effects (font (size 1.27 1.27)))
     )
-    (property "Footprint" "2SB1730" (at 201.93 26.67 0)
+    (property "Footprint" "SamacSys_Parts:2SB1730" (at 201.93 26.67 0)
       (effects (font (size 1.27 1.27)) (justify left) hide)
     )
@@
   )
   (symbol (lib_id "Connector:Conn_01x06_Pin") (at 215.9 113.03 270) (unit 1)
-    (in_bom no) (on_board yes) (dnp no) (fields_autoplaced)
+    (in_bom yes) (on_board yes) (dnp no) (fields_autoplaced)
     (property "Reference" "J5" (at 214.63 109.22 90)
       (effects (font (size 1.27 1.27)))
@@
   (symbol (lib_id "power:+5V") (at 85.09 91.44 0) (unit 1)
     (in_bom yes) (on_board yes) (dnp no) (fields_autoplaced)
-    (property "Reference" "#PWR035" (at 85.09 95.25 0)
+    (property "Reference" "#PWR036" (at 85.09 95.25 0)
       (effects (font (size 1.27 1.27)) hide)
     )
@@
       (project "greenhouse_project_hat"
         (path "/b27d5451-0104-43eb-badd-cec4b3afa639/a0f75671-40a3-4d36-8542-9696f27b0c1b"
-          (reference "#PWR035") (unit 1)
+          (reference "#PWR036") (unit 1)
         )
       )
@@
   )
   (symbol (lib_id "Connector:Conn_01x06_Pin") (at 246.38 113.03 270) (unit 1)
-    (in_bom no) (on_board yes) (dnp no) (fields_autoplaced)
+    (in_bom yes) (on_board yes) (dnp no) (fields_autoplaced)
     (property "Reference" "J7" (at 245.11 109.22 90)
       (effects (font (size 1.27 1.27)))
@@
   )
   (symbol (lib_id "Connector:Conn_01x06_Pin") (at 215.9 132.08 270) (unit 1)
-    (in_bom no) (on_board yes) (dnp no) (fields_autoplaced)
+    (in_bom yes) (on_board yes) (dnp no) (fields_autoplaced)
     (property "Reference" "J6" (at 214.63 128.27 90)
       (effects (font (size 1.27 1.27)))
@@
   )
   (symbol (lib_id "Connector:Conn_01x06_Pin") (at 246.38 133.35 270) (unit 1)
-    (in_bom no) (on_board yes) (dnp no) (fields_autoplaced)
+    (in_bom yes) (on_board yes) (dnp no) (fields_autoplaced)
     (property "Reference" "J8" (at 245.11 129.54 90)
       (effects (font (size 1.27 1.27)))
