File: PCB/screen/greenhouse_project_screen/greenhouse_project_screen.kicad_pcb (KiCad board)
At the start: 2 copper layers, 95.2 x 47 mm, 36 parts, among them IC1 CD74HC14M96, J2 Conn_01x10_Socket, SW1 SW_Push, SW2 SW_Push, SW3 SW_Push, SW4 SW_Push, SW5 SW_Push

Commit message: First production version
Other:
- board text added: "SW4"
